Commit message: Add sensor usb-camera from youbot_description package. A little bit change camera's gazebo.urdf.xacro file. Now it's work fine

File: youbot_description/urdf/sensors/microsoft_lifecam.gazebo.xacro (robot description, xacro)
@@ -6,25 +6,38 @@
 <xacro:macro name="microsoft_lifecam_gazebo" params="name">
   <gazebo reference="${name}_camera">
-    <sensor:camera name="${name}_rgb_frame_sensor">
-      <imageFormat>R8G8B8</imageFormat>
-      <imageSize>1920 1080</imageSize>
-      <hfov>70</hfov>
-      <nearClip>0.01</nearClip>
-      <farClip>5</farClip>
-      <updateRate>20.0</updateRate>
-      <baseline>0.2</baseline>
-      <controller:gazebo_ros_camera name="${name}_rgb_frame_controller" plugin="libgazebo_ros_camera.so">
+    <sensor type="camera" name="camera1">
+      <update_rate>30.0</update_rate>
+      <camera name="head">
+        <horizontal_fov>1.3962634</horizontal_fov>
+        <image>
+          <width>800</width>
+          <height>800</height>
+          <format>R8G8B8</format>
+        </image>
+        <clip>
+          <near>0.02</near>
+          <far>300</far>
+        </clip>
+        <noise>
+          <type>gaussian</type>
+          <mean>0.0</mean>
+          <stddev>0.007</stddev>
+        </noise>
+      </camera>
+      <plugin name="camera_controller" filename="libgazebo_ros_camera.so">
         <alwaysOn>true</alwaysOn>
-        <updateRate>20.0</updateRate>
-        <imageTopicName>/usb_cam/image_raw</imageTopicName>
-        <cameraInfoTopicName>/usb_cam/camera_info</cameraInfoTopicName>
-        <frameName>/${name}_frame</frameName>
-        <distortion_k1>0.00000001</distortion_k1>
-        <distortion_k2>0.00000001</distortion_k2>
-        <distortion_k3>0.00000001</distortion_k3>
-        <distortion_t1>0.00000001</distortion_t1>
-        <distortion_t2>0.00000001</distortion_t2>
-      </controller:gazebo_ros_camera>
-    </sensor:camera>
+        <updateRate>0.0</updateRate>
+        <cameraName>usb_cam</cameraName>
+        <imageTopicName>image_raw</imageTopicName>
+        <cameraInfoTopicName>camera_info</cameraInfoTopicName>
+        <frameName>camera_link</frameName>
+        <hackBaseline>0.07</hackBaseline>
+        <distortionK1>0.0</distortionK1>
+        <distortionK2>0.0</distortionK2>
+        <distortionK3>0.0</distortionK3>
+        <distortionT1>0.0</distortionT1>
+        <distortionT2>0.0</distortionT2>
+      </plugin>
+    </sensor>
   </gazebo>
 </xacro:macro>

File: youbot_description/urdf/sensors/microsoft_lifecam.urdf.xacro (robot description, xacro)
@@ -24,4 +24,5 @@
        <mesh filename="package://youbot_description/meshes/sensors/microsoft_lifecam.dae" scale="0.001 0.001 0.001"/>
       </geometry>
+    <material name="DarkGrey" />
     </visual>
     <collision>
