Commit message: Add checkboard to simulation.

File: youbot_description/urdf/sensors/microsoft_lifecam.urdf.xacro (robot description, xacro)
@@ -26,10 +26,10 @@
     <material name="DarkGrey" />
     </visual>
-    <collision>
+    <!-- <collision>
       <origin xyz="-0.04 -0.0035 -0.031" rpy="${M_PI/2} 0 ${M_PI/2}" />
       <geometry>
         <mesh filename="package://youbot_description/meshes/sensors/microsoft_lifecam.dae" scale="0.001 0.001 0.001"/>
       </geometry>
-    </collision>
+    </collision> -->
   </link>
   <!-- for simulation -->

File: youbot_simulation/urdf/youbot_cam_1.urdf.xacro (robot description, xacro)
@@ -23,4 +23,7 @@
   <xacro:include filename="$(find youbot_description)/urdf/sensors/hokuyo_urg04_laser.urdf.xacro"/>
   <xacro:include filename="$(find youbot_description)/urdf/sensors/microsoft_lifecam.urdf.xacro"/>
+  <!-- checkboard -->
+<xacro:include filename="$(find youbot_simulation)/urdf/checkboard.xacro"/>
+<xacro:include filename="$(find youbot_simulation)/urdf/material.urdf.xacro" />
   <!-- foot for arm-->
   <xacro:youbot_base name="base"/>
@@ -42,3 +45,7 @@
     <origin xyz="-0.048 0 0.001" rpy="0 ${-pi/2} 0" />
   </xacro:microsoft_lifecam>
+  <!-- checkboard -->
+  <xacro:checkboard name="checkboard" parent="plate_link">
+    <origin xyz="0 0.01 0.025" rpy="0 0 ${-pi/2} " />
+  </xacro:checkboard>
 </robot>
